File: pcb/raw.kicad_pcb (KiCad board)
At the start: 2 copper layers, 249.4 x 123.5 mm, 223 parts

Commit message: Pin remapping for a more elegant layout
Connections:
- D11 pad 2: P14 -> P15
- D12 pad 2: P15 -> P20
- D14 pad 2: P14 -> P15
- D15 pad 2: P15 -> P20
- D19 pad 2: P7 -> P9
- D2 pad 2: P14 -> P15
- D21 pad 2: P5 -> P2
- D22 pad 2: P7 -> P9
- D24 pad 2: P5 -> P2
- D25 pad 2: P7 -> P9
- D27 pad 2: P5 -> P2
- D28 pad 2: P7 -> P9
- D3 pad 2: P15 -> P20
- D30 pad 2: P5 -> P2
- D31 pad 2: P7 -> P9
- D33 pad 2: P5 -> P2
- D34 pad 2: P8 -> P19
- D35 pad 2: P8 -> P19
- D36 pad 2: P8 -> P19
- D5 pad 2: P14 -> P15
- D6 pad 2: P15 -> P20
- D8 pad 2: P14 -> P15
- D9 pad 2: P15 -> P20
- L1 pad 4: P9 -> P18
- L1 pad 44: P9 -> P18
- P10 pad 1: P2 -> P7
- P11 pad 1: P3 -> P8
- P12 pad 1: P3 -> P8
- P13 pad 1: P4 -> P1
- P14 pad 1: P4 -> P1
- P16 pad 1: P7 -> P9
- P17 pad 1: P1 -> P4
- P19 pad 1: P5 -> P2
- P2 pad 1: P1 -> P4
- P20 pad 1: P1 -> P4
- P21 pad 1: P19 -> P3
- P22 pad 1: P0 -> P5
- P23 pad 1: P0 -> P5
- P24 pad 1: P2 -> P7
- P25 pad 1: P2 -> P7
- P26 pad 1: P3 -> P8
- P27 pad 1: P3 -> P8
- P28 pad 1: P4 -> P1
- P29 pad 1: P4 -> P1
- P3 pad 1: P14 -> P15
- P30 pad 1: P8 -> P19
- P31 pad 1: P20 -> P21
- P32 pad 1: P21 -> P0
- P4 pad 1: P15 -> P20
- P5 pad 1: P1 -> P4
- P6 pad 1: P19 -> P3
- P7 pad 1: P0 -> P5
- P8 pad 1: P0 -> P5
- P9 pad 1: P2 -> P7
- S1 pad 2: P1 -> P4
- S10 pad 2: P0 -> P5
- S100 pad 1: P2 -> P7
- S101 pad 1: P2 -> P7
- S102 pad 1: P2 -> P7
- S103 pad 1: P3 -> P8
- S104 pad 1: P3 -> P8
- S105 pad 1: P3 -> P8
- S106 pad 1: P3 -> P8
- S107 pad 1: P3 -> P8
- S108 pad 1: P3 -> P8
- S109 pad 1: P3 -> P8
- S11 pad 2: P0 -> P5
- S110 pad 1: P3 -> P8
- S111 pad 1: P3 -> P8
- S112 pad 1: P4 -> P1
- S113 pad 1: P4 -> P1
- S114 pad 1: P4 -> P1
- S115 pad 1: P4 -> P1
- S116 pad 1: P4 -> P1
- S117 pad 1: P4 -> P1
- S118 pad 1: P4 -> P1
- S119 pad 1: P4 -> P1
- S12 pad 2: P0 -> P5
- S120 pad 1: P4 -> P1
- S121 pad 1: P1 -> P4
- S122 pad 1: P1 -> P4
- S123 pad 1: P1 -> P4
- S124 pad 1: P0 -> P5
- S125 pad 1: P0 -> P5
- S126 pad 1: P0 -> P5
- S127 pad 1: P2 -> P7
- S128 pad 1: P2 -> P7
- S129 pad 1: P2 -> P7
- S13 pad 2: P0 -> P5
- S130 pad 1: P3 -> P8
- S131 pad 1: P3 -> P8
- S132 pad 1: P3 -> P8
- S133 pad 1: P4 -> P1
- S134 pad 1: P4 -> P1
- S135 pad 1: P4 -> P1
- S136 pad 2: P2 -> P7
- S137 pad 2: P2 -> P7
- S138 pad 2: P2 -> P7
- S139 pad 2: P3 -> P8
- S14 pad 2: P0 -> P5
- S140 pad 2: P3 -> P8
- S141 pad 2: P3 -> P8
- S142 pad 2: P4 -> P1
- S143 pad 2: P4 -> P1
- S144 pad 2: P4 -> P1
- S145 pad 2: P4 -> P1
- S146 pad 2: P4 -> P1
- S147 pad 2: P4 -> P1
- S148 pad 2: P2 -> P7
- S149 pad 2: P2 -> P7
- S15 pad 2: P0 -> P5
- S150 pad 2: P2 -> P7
- S16 pad 2: P0 -> P5
- S17 pad 2: P0 -> P5
- S18 pad 2: P0 -> P5
- S19 pad 2: P2 -> P7
- S2 pad 2: P1 -> P4
- S20 pad 2: P2 -> P7
- S21 pad 2: P2 -> P7
- S22 pad 2: P2 -> P7
- S23 pad 2: P2 -> P7
- S24 pad 2: P2 -> P7
- S25 pad 2: P2 -> P7
- S26 pad 2: P2 -> P7
- S27 pad 2: P2 -> P7
- S28 pad 2: P3 -> P8
- S29 pad 2: P3 -> P8
- S3 pad 2: P1 -> P4
- S30 pad 2: P3 -> P8
- S31 pad 2: P3 -> P8
- S32 pad 2: P3 -> P8
- S33 pad 2: P3 -> P8
- S34 pad 2: P3 -> P8
- S35 pad 2: P3 -> P8
- S36 pad 2: P3 -> P8
- S37 pad 2: P4 -> P1
- S38 pad 2: P4 -> P1
- S39 pad 2: P4 -> P1
- S4 pad 2: P1 -> P4
- S40 pad 2: P4 -> P1
- S41 pad 2: P4 -> P1
- S42 pad 2: P4 -> P1
- S43 pad 2: P4 -> P1
- S44 pad 2: P4 -> P1
- S45 pad 2: P4 -> P1
- S46 pad 2: P1 -> P4
- S47 pad 2: P1 -> P4
- S48 pad 2: P1 -> P4
- S49 pad 2: P0 -> P5
- S5 pad 2: P1 -> P4
- S50 pad 2: P0 -> P5
- S51 pad 2: P0 -> P5
- S52 pad 2: P2 -> P7
- S53 pad 2: P2 -> P7
- S54 pad 2: P2 -> P7
- S55 pad 2: P3 -> P8
- S56 pad 2: P3 -> P8
- S57 pad 2: P3 -> P8
- S58 pad 2: P4 -> P1
- S59 pad 2: P4 -> P1
- S6 pad 2: P1 -> P4
- S60 pad 2: P4 -> P1
- S61 pad 2: P2 -> P7
- S62 pad 2: P2 -> P7
- S63 pad 2: P2 -> P7
- S64 pad 2: P3 -> P8
- S65 pad 2: P3 -> P8
- S66 pad 2: P3 -> P8
- S67 pad 2: P4 -> P1
- S68 pad 2: P4 -> P1
- S69 pad 2: P4 -> P1
- S7 pad 2: P1 -> P4
- S70 pad 2: P4 -> P1
- S71 pad 2: P4 -> P1
- S72 pad 2: P4 -> P1
- S73 pad 2: P2 -> P7
- S74 pad 2: P2 -> P7
- S75 pad 2: P2 -> P7
- S76 pad 1: P1 -> P4
- S77 pad 1: P1 -> P4
- S78 pad 1: P1 -> P4
- S79 pad 1: P1 -> P4
- S8 pad 2: P1 -> P4
- S80 pad 1: P1 -> P4
- S81 pad 1: P1 -> P4
- S82 pad 1: P1 -> P4
- S83 pad 1: P1 -> P4
- S84 pad 1: P1 -> P4
- S85 pad 1: P0 -> P5
- S86 pad 1: P0 -> P5
- S87 pad 1: P0 -> P5
- S88 pad 1: P0 -> P5
- S89 pad 1: P0 -> P5
- S9 pad 2: P1 -> P4
- S90 pad 1: P0 -> P5
- S91 pad 1: P0 -> P5
- S92 pad 1: P0 -> P5
- S93 pad 1: P0 -> P5
- S94 pad 1: P2 -> P7
- S95 pad 1: P2 -> P7
- S96 pad 1: P2 -> P7
- S97 pad 1: P2 -> P7
- S98 pad 1: P2 -> P7
- S99 pad 1: P2 -> P7
- T1 pad 1: RAWER -> RAW
- T1 pad 2: RAW -> RAWER
