File: pcb/absolem.kicad_pcb (KiCad board)
At the start: 2 copper layers, 249.4 x 123.5 mm, 223 parts

Commit message: First PCB release candidate
Parts:
- added GBACK: LOGO, LOGO, F.Cu at (116.8, 40.6)
- added GFRONT: LOGO, LOGO, F.Cu at (116.8, 17.8)
Routing:
- net P7: track 461.8 -> 475.5 mm
- net P1: track 394.8 -> 408.3 mm
- net P2: track 160.1 -> 163.5 mm
- net P4: track 388.3 -> 387.4 mm
- net P3: track 259.7 -> 260.5 mm
- net GND: track 98.4 -> 97.8 mm

Commit message: Easter eggs + minor metadata fix
Other:
- board text added: "Drink me!"
- board text added: "Eat me!"
